File: PCB/reQUAD.kicad_pcb (KiCad board)
At the start: 2 copper layers, 49.5 x 16.5 mm, 10 parts, among them J1 Model_100_System_BUS, U1 7474, U2 7402, U4 74573, U5 628128

Commit message: v002
Other:
- board text added: "v002"
- board text removed: "v001"

Commit message: v003
Parts:
- added D2: BAV70, 000_LOCAL:SOT-23, F.Cu at (138.8, 105.0)
- added D3: BAV70, 000_LOCAL:SOT-23, F.Cu at (127.8, 105.1)
- added U6: 74LVC2G14, 000_LOCAL:SC-74-6_1.5x2.9mm_P0.95mm, F.Cu at (131.7, 105.1)
- D1: value BAV70S -> BAV70; footprint 000_LOCAL:SOT-363_SC-70-6 -> 000_LOCAL:SOT-23
- moved C1 14.8 mm to (145.3, 97.8), turned to 90 degrees
- moved D1 14.2 mm to (142.6, 105.0), turned to 90 degrees
- moved R1 2.16 mm to (135.2, 99.0)
- moved C2 1.59 mm to (135.2, 102.2)
Connections:
- C2 pad 1: /FLOP_CLR -> Net-(C2-Pad1)
- D1 pad 1: VDD -> /RAMRST
- D1 pad 2: /RAMRST -> VCC
- D1 pad 3: /RAMRST -> /VMEM
- J1 pad 1: VDD -> VCC
- J1 pad 40: VDD -> VCC
- R1 pad 1: VDD -> VCC
- R1 pad 2: /FLOP_CLR -> Net-(C2-Pad1)
- U1 pad 10: VDD -> VCC
- U1 pad 14: VDD -> VCC
- U1 pad 4: VDD -> VCC
- U2 pad 14: VDD -> VCC
- U4 pad 20: VDD -> VCC
Routing:
- net VCC: track 0.00 -> 108.9 mm, vias 0 -> 6
- net VDD: track 97.8 -> 0.00 mm, vias 4 -> 0
- net /VMEM: track 22.1 -> 8.60 mm
- net Net-(C2-Pad1): track 0.00 -> 12.2 mm, vias 0 -> 2
- net /RAMRST: track 3.19 -> 14.1 mm, vias 0 -> 1
- net /FLOP_CLR: track 10.4 -> 14.2 mm, vias 0 -> 2
- net Net-(U6-Pad3): track 0.00 -> 3.39 mm
- net /AD0: track 62.7 -> 66.0 mm
- net /B0: track 24.2 -> 21.2 mm
- net /~{WR}: track 14.3 -> 17.3 mm
- net /FLOP_CLK: track 13.0 -> 10.7 mm
- net /AD7: track 13.8 -> 15.6 mm
- net /A15: track 14.1 -> 15.5 mm
- net /A8: track 22.6 -> 21.2 mm
- net /B1: track 18.9 -> 20.3 mm, vias 2 -> 0
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Other:
- board text added: "Based on QUADv4 by Steve Adolph"
- board text added: "b.kenyon.w@gmail.com"
- board text added: "v003"
- board text removed: "Circuit: Steve Adolph"
- board text removed: "PCB: b.kenyon.w@gmail.com"
- board text removed: "v002"

Commit message: v004
Parts:
- removed C2: 1uF, 000_LOCAL:C_0805
- removed D2, D3: BAV70, 000_LOCAL:SOT-23
- removed R1: 340K, 000_LOCAL:R_0805
- removed U6: 74LVC2G14, 000_LOCAL:SC-74-6_1.5x2.9mm_P0.95mm
- D1: value BAV70 -> BAV70S; footprint 000_LOCAL:SOT-23 -> 000_LOCAL:SOT-363_SC-70-6
- moved D1 7.25 mm to (135.4, 104.6), turned to 0 degrees
Connections:
- C1 pad 1: /VMEM -> VMEM
- D1 pad 1: /RAMRST -> VCC
- D1 pad 2: VCC -> /RAMRST
- D1 pad 3: /VMEM -> /RAMRST
- U1 pad 1: /FLOP_CLR -> (no net)
- U1 pad 10: VCC -> (no net)
- U1 pad 13: /FLOP_CLR -> (no net)
- U1 pad 14: VCC -> VMEM
- U1 pad 4: VCC -> (no net)
- U5 pad 8: /VMEM -> VMEM
Routing:
- net VCC: track 108.9 -> 69.5 mm, vias 6 -> 5
- net VMEM: track 0.00 -> 26.3 mm, vias 0 -> 2
- net /FLOP_CLR: track 14.2 -> 0.00 mm, vias 2 -> 0
- net Net-(C2-Pad1): track 12.2 -> 0.00 mm, vias 2 -> 0
- net /VMEM: track 8.60 -> 0.00 mm
- net /RAMRST: track 14.1 -> 7.68 mm, vias 1 -> 0
- net Net-(U6-Pad3): track 3.39 -> 0.00 mm
- net /AD0: track 66.0 -> 63.3 mm
- net /AD7: track 15.6 -> 13.8 mm
- net /B1: track 20.3 -> 22.0 mm, vias 0 -> 2
- net /A8: track 21.2 -> 22.6 mm
- net /B0: track 21.2 -> 20.1 mm
- net GND: vias 5 -> 13
Other:
- board text added: "v004"
- board text removed: "v003"

Commit message: v005
Parts:
- D1: value BAV70S -> BAV70; footprint 000_LOCAL:SOT-363_SC-70-6 -> 000_LOCAL:SOT-363_symmetric
- U1: value 7474 -> 74LVC2G79; footprint 000_LOCAL:SOIC-14_3.9x8.7mm_P1.27mm -> 000_LOCAL:VSSOP-8_2.3x2mm_P0.5mm
- U2: value 7402 -> 74AC02; footprint 000_LOCAL:SOIC-14_3.9x8.7mm_P1.27mm -> 000_LOCAL:TSSOP-14_4.4x5mm_P0.65mm
- U4: value 74573 -> 74AC573
- moved U2 5.75 mm to (134.8, 98.1)
- moved U1 4.67 mm to (133.1, 102.5)
- moved D1 2.76 mm to (137.1, 102.4)
- moved C1 0.91 mm to (144.4, 98.0)
Connections:
- U1 pad 1: (no net) -> /FLOP_CLK
- U1 pad 3: /FLOP_CLK -> /B1
- U1 pad 4: (no net) -> GND
- U1 pad 5: /B0 -> /FLOP_CLK
- U1 pad 6: (no net) -> /AD1
- U1 pad 7: GND -> /B0
- U1 pad 8: (no net) -> VMEM
Routing:
- net VMEM: track 26.3 -> 14.3 mm, vias 2 -> 0
- net /AD0: track 63.3 -> 57.6 mm, vias 4 -> 2
- net /~{Y0}: track 5.81 -> 11.1 mm, vias 1 -> 2
- net /A15: track 15.5 -> 20.7 mm
- net /U5_CE2: track 5.43 -> 10.6 mm
- net /RESET: track 11.4 -> 6.70 mm
- net /B1: track 22.0 -> 17.8 mm, vias 2 -> 0
- net /B0: track 20.1 -> 16.0 mm
- net /~{WR}: track 17.1 -> 20.2 mm, vias 2 -> 1
- net VCC: track 69.5 -> 66.6 mm
- net /RAMRST: track 7.68 -> 10.4 mm, vias 0 -> 1
- net /FLOP_CLK: track 10.7 -> 8.66 mm
- net /ALE: track 39.8 -> 38.3 mm
- net Net-(U2-Pad1): track 6.74 -> 5.31 mm, vias 2 -> 0
- net /AD1: track 64.2 -> 63.3 mm
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Other:
- board text added: "v005"
- board text removed: "v004"

Commit message: v006
Parts:
- moved U5 4.02 mm to (150.0, 100.0)
- moved C1 3.84 mm to (141.1, 100.0)
- moved U4 3.18 mm to (164.0, 100.0)
- moved D1 1.65 mm to (138.6, 103.2)
- moved U2 1.27 mm to (136.0, 98.1)
- moved U1 1.23 mm to (134.1, 103.2)
Routing:
- net VCC: track 66.6 -> 98.8 mm, vias 5 -> 3
- net /AD1: track 63.3 -> 49.4 mm, vias 4 -> 6
- net /AD0: track 57.6 -> 46.5 mm, vias 2 -> 6
- net /A2: track 4.14 -> 12.2 mm
- net /IO~{M}: track 27.6 -> 20.6 mm, vias 2 -> 1
- net /A8: track 22.6 -> 28.6 mm
- net /~{RD}: track 25.2 -> 19.6 mm, vias 2 -> 1
- net /U5_CE2: track 10.6 -> 5.17 mm
- net /B0: track 16.0 -> 10.9 mm
- net /AD5: track 15.7 -> 20.7 mm, vias 3 -> 2
- net /AD3: track 18.1 -> 22.4 mm, vias 3 -> 2
- net VMEM: track 14.3 -> 10.0 mm
- net /A3: track 4.08 -> 8.19 mm
- net /A15: track 20.7 -> 16.7 mm
- net /ALE: track 38.3 -> 34.5 mm, vias 1 -> 0
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Other:
- board text added: "v006"
- board text removed: "v005"

Commit message: v007
Parts:
- D1: footprint 000_LOCAL:SOT-363_symmetric -> 000_LOCAL:SOT-23
- U1: footprint 000_LOCAL:VSSOP-8_2.3x2mm_P0.5mm -> 000_LOCAL:SSOP-8
- moved D1 1.28 mm to (139.8, 103.4), turned to 90 degrees
- moved U1 0.63 mm to (134.8, 103.2)
Connections:
- D1 pad 1: VCC -> (no net)
- D1 pad 2: /RAMRST -> VCC
- D1 pad 3: /RAMRST -> VMEM
- J1 pad 19: /RAMRST -> VMEM
- U2 pad 14: VCC -> VMEM
Routing:
- net VCC: track 98.8 -> 63.3 mm, vias 3 -> 2
- net VMEM: track 10.0 -> 30.9 mm, vias 0 -> 2
- net /RAMRST: track 11.4 -> 0.00 mm
- net /ALE: track 34.5 -> 29.4 mm, vias 0 -> 2
- net /AD6: track 21.5 -> 25.6 mm, vias 2 -> 1
- net /AD1: track 49.4 -> 45.8 mm, vias 6 -> 4
- net /B1: track 15.0 -> 11.9 mm
- net /FLOP_CLK: track 9.69 -> 10.8 mm
- net /AD0: track 46.5 -> 46.1 mm, vias 6 -> 4
- net GND: vias 16 -> 4
Other:
- board text added: "legs this side"
- board text added: "v007"
- board text removed: "v006"
