File: PCB/reQUAD.kicad_sch (KiCad schematic)
At the start: 10 parts, among them J1 Model_100_System_BUS, U1 7474, U2 7402, U3 74LVC2G14, U4 74573, U5 628128

Commit message: v002
Parts:
- removed U3: 74LVC2G14, symbol 000_LOCAL:74LVC2G14
Connections:
- net FLOP_CLR: now also C2.1, R1.2
Other:
- moved on the sheet: C2, R1, U1C, U2E

Commit message: v003
Parts:
- removed D1: BAV70S, 000_LOCAL:SOT-363_SC-70-6, symbol 000_LOCAL:BAV70S
- added D1, D2, D3: BAV70, 000_LOCAL:SOT-23, symbol 000_LOCAL:BAV70
- added U6: 74HC2G14GV, 000_LOCAL:SC-74-6_1.5x2.9mm_P0.95mm, symbol 000_LOCAL:74LVC2G14
Connections:
- net FLOP_CLR: now also U6.4; no longer C2.1, R1.2
- net GND: now also U6.2 (GND), U6.2 (GND)
- net RAMRST: now also D1.1 (A), D2.3 (K)
- net VMEM: now also D1.3 (K)
- net VDD renamed VCC
- net VCC: now also D1.2 (A), D2.1 (A), D3.3 (K), U6.5 (VCC), U6.5 (VCC)
- new net: C2.1, D3.2 (A), R1.2, U6.1
- new net: U6.3, U6.6
- no-connect marks 9 -> 10
Other:
- moved on the sheet: C2, R1, U1C, U2E

Commit message: v004
Parts:
- removed C2: 1uF, 000_LOCAL:C_0805, symbol 000_LOCAL:C_Small
- removed D3: BAV70, 000_LOCAL:SOT-23, symbol 000_LOCAL:BAV70
- removed R1: 340K, 000_LOCAL:R_0805, symbol 000_LOCAL:R_Small
- removed U6: 74HC2G14GV, 000_LOCAL:SC-74-6_1.5x2.9mm_P0.95mm, symbol 000_LOCAL:74LVC2G14
- D1: value BAV70 -> BAV70S; footprint 000_LOCAL:SOT-23 -> 000_LOCAL:SOT-363_SC-70-6; symbol 000_LOCAL:BAV70 -> 000_LOCAL:BAV70S
- D1: renamed from D2; value BAV70 -> BAV70S; footprint 000_LOCAL:SOT-23 -> 000_LOCAL:SOT-363_SC-70-6; symbol 000_LOCAL:BAV70 -> 000_LOCAL:BAV70S
Connections:
- net RAMRST: now also D1.2 (A); no longer D1.1 (A)
- net VCC: now also D1.1 (A), D1.5 (A); no longer D1.1 (A), D1.2 (A), U1.10 (~{S}), U1.14 (VCC), U1.4 (~{S})
- net VMEM: now also D1.6 (K), U1.14 (VCC); no longer D1.3 (K)
- net FLOP_CLR: no longer names the net of U1.1 (~{R})
- net FLOP_CLR: no longer U1.13 (~{R})
- no-connect marks 10 -> 13
Other:
- moved on the sheet: U1A, U1B, U1C, U2E

Commit message: v005
Parts:
- removed unit 3 of U1
- added unit 3 of U1
- D1: value BAV70S -> BAV70; footprint 000_LOCAL:SOT-363_SC-70-6 -> 000_LOCAL:SOT-363_symmetric
- U1: value 7474 -> 74LVC2G79; footprint 000_LOCAL:SOIC-14_3.9x8.7mm_P1.27mm -> 000_LOCAL:VSSOP-8_2.3x2mm_P0.5mm; symbol 000_LOCAL:7474 -> 000_LOCAL:74LVC2G79
- U2: value 7402 -> 74AC02; footprint 000_LOCAL:SOIC-14_3.9x8.7mm_P1.27mm -> 000_LOCAL:TSSOP-14_4.4x5mm_P0.65mm
- U4: value 74573 -> 74AC573
Connections:
- net AD1: now also U1.6 (D); no longer U1.12 (D)
- net B0: now also U1.7 (Q); no longer U1.5 (Q)
- net B1: now also U1.3 (Q); no longer U1.9 (Q)
- net FLOP_CLK: now also U1.1 (C), U1.5 (C); no longer U1.11 (C), U1.3 (C)
- net GND: now also U1.4 (GND)
- net VMEM: now also U1.8 (VCC)
- no-connect marks 13 -> 7
Other:
- note removed: "74AC02"
- note removed: "74AC573"
- note removed: "74AC74"
- moved on the sheet: C1, D1A, D1B, U2A, U2B, U2C, U2D, U2E

Commit message: v007
Parts:
- removed unit 2 of D1
- D1: footprint 000_LOCAL:SOT-363_symmetric -> 000_LOCAL:SOT-23; symbol 000_LOCAL:BAV70S -> 000_LOCAL:BAV70
- U1: footprint 000_LOCAL:VSSOP-8_2.3x2mm_P0.5mm -> 000_LOCAL:SSOP-8
- U1: footprint (none) -> 000_LOCAL:SSOP-8
Connections:
- net VCC: now also D1.2 (A); no longer D1.1 (A), U2.14 (VCC)
- net VMEM: now also D1.3 (K), J1.19 (RAMRST), U2.14 (VCC); no longer D1.6 (K)
- removed net RAMRST: D1.2 (A), J1.19 (RAMRST)
- no-connect marks 7 -> 6
Other:
- moved on the sheet: C1, D1, U1A, U1B, U1C, U2A, U2B, U2C, U2D, U2E, U5
