File: PCB/reQUAD_018.kicad_sch (KiCad schematic)
At the start: 12 parts, among them J1 Model_100_System_BUS, U1 AS6C1008, U2 74x573, U3 74x2G79, U4 74x02

Commit message: make v020 main even though not tested yet
Parts:
- removed BT1: Keystone_3031, 000_LOCAL:Keystone_3031, symbol 000_LOCAL:Battery_Cell
- removed C4: 220u, 000_LOCAL:CP_EIA-6032-28, symbol 000_LOCAL:C
- removed DA1: BAV756S, 000_LOCAL:SOT-363, symbol 000_LOCAL:BAV756S
- added DA1: BAV70S, 000_LOCAL:SOT-363_symmetric, symbol 000_LOCAL:BAV70S
- U1: footprint 000_LOCAL:TSOP32-dual -> 000_LOCAL:TSOP32-14mm
Connections:
- net A0: now also U1.20 (A0); no longer U1.16 (A4)
- net A1: now also U1.19 (A1); no longer U1.15 (A5)
- net A11: now also U1.1 (A11); no longer U1.2 (A9)
- net A12: now also U1.12 (A12); no longer U1.11 (A14)
- net A13: now also U1.4 (A13); no longer U1.1 (A11)
- net A14: now also U1.11 (A14); no longer U1.12 (A12)
- net A2: now also U1.18 (A2); no longer U1.14 (A6)
- net A3: now also U1.17 (A3); no longer U1.13 (A7)
- net A4: now also U1.16 (A4); no longer U1.17 (A3)
- net A5: now also U1.15 (A5); no longer U1.18 (A2)
- net A6: now also U1.14 (A6); no longer U1.19 (A1)
- net A7: now also U1.13 (A7); no longer U1.20 (A0)
- net A8: now also U1.3 (A8); no longer U1.4 (A13)
- net A9: now also U1.2 (A9); no longer U1.3 (A8)
- net BANK_LATCH: now also U4.4; no longer U4.1
- net BUS_A15: now also U4.8, U4.9; no longer U4.11, U4.12
- net RAM_CE2: now also U4.13; no longer U4.10
- net RAM_RST: now also DA1.2 (A), DA1.3 (K)
- net RESET: now also U4.12; no longer U4.8
- net VBUS: now also DA1.1 (A), DA1.5 (A)
- net VMEM: now also DA1.6 (K)
- net ~{WR}: now also U4.3; no longer U4.5
- net ~{Y0}: now also U4.2; no longer U4.6
- new net: U4.1, U4.5, U4.6
- new net: U4.10, U4.11
- no-connect marks 6 -> 7
Other:
- note added: "Disable internal RAM"
- moved on the sheet: C1, C2, C3, U3C, U4A, U4B, U4C, U4D, U4E
